File: KiCad/Prototype/project.sch (KiCad schematic (older format))
At the start: 43 parts, among them J1 Barrel_Jack, J2 USB_B, J3 ICSP, J4 BANK 0..7, J5 BANK 8..15, Q1 PMOS, SW1 RESET, U1 LP2985-3.3, U2 LMV358, U3 NCP1117-1.5, U4 ATMEGA32U4-AU, Y1 16 Mhz

Commit message: mainly finished schematic
Parts:
- removed JP?: PULL, Jumper:SolderJumper-3_P1.3mm_Bridged12_Pad1.0x1.5mm, symbol Jumper:Jumper_3_Bridged12
- added D? (x3): 1N914WT, Diode_SMD:D_SOD-523, symbol Diode:1N914WT
- added D? (x6): BAV70, Package_TO_SOT_SMD:SOT-23, symbol Diode:BAV70
- added J?: MIDI IN, symbol Connector:DIN-5_180degree
- added J?: MIDI OUT, symbol Connector:DIN-5_180degree
- added J?: POT 5, Connector_JST:JST_XH_B03B-XH-A_1x03_P2.50mm_Vertical, symbol Connector:Conn_01x03_Male
- added J?: POT 6, Connector_JST:JST_XH_B03B-XH-A_1x03_P2.50mm_Vertical, symbol Connector:Conn_01x03_Male
- added J?: POT 3, Connector_JST:JST_XH_B03B-XH-A_1x03_P2.50mm_Vertical, symbol Connector:Conn_01x03_Male
- added J?: POT 4, Connector_JST:JST_XH_B03B-XH-A_1x03_P2.50mm_Vertical, symbol Connector:Conn_01x03_Male
- added J?: POT 1, Connector_JST:JST_XH_B03B-XH-A_1x03_P2.50mm_Vertical, symbol Connector:Conn_01x03_Male
- added J?: POT 2, Connector_JST:JST_XH_B03B-XH-A_1x03_P2.50mm_Vertical, symbol Connector:Conn_01x03_Male
- added J?: PRESSURE, Connector_IDC:IDC-Header_2x06_P2.54mm_Vertical, symbol Connector_Generic:Conn_02x06_Odd_Even
- added Q?: MMBT3904, Package_TO_SOT_SMD:SOT-23, symbol Transistor_BJT:MMBT3904
- added R? (x4): 220, symbol Device:R
- added R?: 10k, symbol Device:R
- added R?: 270, symbol Device:R
- added R?: 4k7, symbol Device:R
- added RN?: 10k, symbol Device:R_Pack06
- added U?: 6N138, symbol Isolator:6N138
- added U?: 74HC04, symbol 74xx:74HC04
- J?: value AudioJack3_Ground -> EXPRESSION
- J?: value AudioJack2_Ground -> SUSTAIN
- J?: value POTMETER 1 -> POT 7
- J?: value POTMETER 2 -> POT 8
Connections:
- net +5V: now also R?.1, R?.2, U?.8 (VCC)
- net ADC10: now also D?.1 (K), D?.1 (K), D?.3 (K), D?.3 (K), D?.3 (K), D?.3 (K), D?.3 (K), D?.3 (K)
- net AMUX0: now also R?.2
- net AMUX1: now also R?.2
- net AMUX10: now also J?.3 (Pin_3)
- net AMUX11: now also J?.3 (Pin_3)
- net AMUX12: now also J?.3 (Pin_3)
- net AMUX13: now also J?.3 (Pin_3)
- net AMUX14: now also J?.3 (Pin_3)
- net AMUX15: now also J?.3 (Pin_3)
- net AMUX2: now also J?.1 (Pin_1)
- net AMUX3: now also J?.3 (Pin_3)
- net AMUX4: now also J?.5 (Pin_5)
- net AMUX5: now also J?.7 (Pin_7)
- net AMUX6: now also J?.9 (Pin_9)
- net AMUX7: now also J?.11 (Pin_11)
- net AMUX8: now also J?.3 (Pin_3); no longer J?.3 (Pin_3)
- net AMUX9: now also J?.3 (Pin_3); no longer J?.3 (Pin_3)
- net GND: now also J?.1 (Pin_1), J?.1 (Pin_1), J?.S, J?.S, J?.1 (Pin_1), J?.1 (Pin_1), J?.1 (Pin_1), J?.1 (Pin_1), J?.1 (Pin_1), J?.1 (Pin_1), J?.2, Q?.2 (E), RN?.1 (R1.1), RN?.2 (R2.1), RN?.3 (R3.1), RN?.4 (R4.1), RN?.5 (R5.1), RN?.6 (R6.1), U?.5 (GND)
- net RXD: now also R?.1, U?.6 (VO2)
- net TXD: now also U?.1
- net at J?.R: now also R?.1
- net at J?.T: now also D?.2 (A)
- net at J?.T: now also D?.2 (A), R?.1
- new net: J?.4, R?.1
- new net: D?.2 (A), J?.5, U?.3 (C2)
- new net: J?.4, R?.2
- new net: J?.5, R?.1
- new net: D?.1 (K), R?.2, U?.2 (C1)
- new net: R?.2, U?.2
- new net: Q?.1 (B), R?.1
- new net: Q?.3 (C), R?.2
- new net: D?.1 (A), J?.2 (Pin_2) (x3)
- new net: D?.2 (A), J?.2 (Pin_2) (x3)
- new net: D?.1 (A), J?.10 (Pin_10), RN?.11 (R2.2)
- new net: D?.2 (A), J?.12 (Pin_12), RN?.12 (R1.2)
- new net: D?.1 (A), J?.2 (Pin_2), RN?.7 (R6.2)
- new net: D?.2 (A), J?.4 (Pin_4), RN?.8 (R5.2)
- new net: D?.1 (A), J?.6 (Pin_6), RN?.9 (R4.2)
- new net: D?.2 (A), J?.8 (Pin_8), RN?.10 (R3.2)
- no-connect marks 4 -> 5
Other:
- note added: "Analog input demultiplexers"
- note added: "MIDI in/out"
- note added: "Pedal inputs"
- note added: "Potmeter inputs"
- note added: "Pressure sensor inputs"
- moved on the sheet: D?, J4, J5, J?, U?

Commit message: more footprints
Parts:
- J3: footprint (none) -> Connector_IDC:IDC-Header_2x03_P2.54mm_Vertical
- RN?: footprint (none) -> Resistor_SMD:R_Cat16-8; symbol Device:R_Pack06 -> Device:R_Pack08
- U? (x4): footprint (none) -> Package_SO:TSSOP-16_4.4x5mm_P0.65mm
Connections:
- net at D?.1 (A), J?.10 (Pin_10): now also RN?.15 (R2.2); no longer RN?.11 (R2.2)
- net at D?.2 (A), J?.12 (Pin_12): now also RN?.16 (R1.2); no longer RN?.12 (R1.2)
- net at D?.1 (A), J?.2 (Pin_2): now also RN?.11 (R6.2); no longer RN?.7 (R6.2)
- net at D?.2 (A), J?.4 (Pin_4): now also RN?.12 (R5.2); no longer RN?.8 (R5.2)
- net at D?.1 (A), J?.6 (Pin_6): now also RN?.13 (R4.2); no longer RN?.9 (R4.2)
- net at D?.2 (A), J?.8 (Pin_8): now also RN?.14 (R3.2); no longer RN?.10 (R3.2)
Changed lines of the file:
@@
 F 0 "J3" H 9800 1817 50  0000 C CNN
 F 1 "ICSP" H 9800 1726 50  0000 C CNN
-F 2 "" H 9750 1500 50  0001 C CNN
+F 2 "Connector_IDC:IDC-Header_2x03_P2.54mm_Vertical" H 9750 1500 50  0001 C CNN
 F 3 "~" H 9750 1500 50  0001 C CNN
 	1    9750 1500
@@
 F 0 "U?" H 2350 9000 50  0000 C CNN
 F 1 "74LS138" H 2350 8900 50  0000 C CNN
-F 2 "" H 2150 8450 50  0001 C CNN
+F 2 "Package_SO:TSSOP-16_4.4x5mm_P0.65mm" H 2150 8450 50  0001 C CNN
 F 3 "http://www.ti.com/lit/gpn/sn74LS138" H 2150 8450 50  0001 C CNN
 	1    2150 8450
@@
 F 0 "U?" H 2350 7150 50  0000 C CNN
 F 1 "74LS138" H 2350 7050 50  0000 C CNN
-F 2 "" H 2150 6600 50  0001 C CNN
+F 2 "Package_SO:TSSOP-16_4.4x5mm_P0.65mm" H 2150 6600 50  0001 C CNN
 F 3 "http://www.ti.com/lit/gpn/sn74LS138" H 2150 6600 50  0001 C CNN
 	1    2150 6600
@@
 F 0 "U?" H 5800 9000 50  0000 C CNN
 F 1 "74LS238" H 5800 8900 50  0000 C CNN
-F 2 "" H 5600 8450 50  0001 C CNN
+F 2 "Package_SO:TSSOP-16_4.4x5mm_P0.65mm" H 5600 8450 50  0001 C CNN
 F 3 "http://www.ti.com/lit/gpn/sn74LS138" H 5600 8450 50  0001 C CNN
 	1    5600 8450
@@
 F 0 "U?" H 5800 7150 50  0000 C CNN
 F 1 "74LS238" H 5800 7050 50  0000 C CNN
-F 2 "" H 5600 6600 50  0001 C CNN
+F 2 "Package_SO:TSSOP-16_4.4x5mm_P0.65mm" H 5600 6600 50  0001 C CNN
 F 3 "http://www.ti.com/lit/gpn/sn74LS138" H 5600 6600 50  0001 C CNN
 	1    5600 6600
@@
 $EndComp
 $Comp
-L Device:R_Pack06 RN?
+L Device:R_Pack08 RN?
 U 1 1 5F26B56E
-P 13700 7100
-F 0 "RN?" H 13988 7146 50  0000 L CNN
-F 1 "10k" H 13988 7055 50  0000 L CNN
-F 2 "" V 14075 7100 50  0001 C CNN
-F 3 "~" H 13700 7100 50  0001 C CNN
-	1    13700 7100
-	1    0    0    -1
-$EndComp
+P 13800 7100
+F 0 "RN?" H 14200 7150 50  0000 L CNN
+F 1 "10k" H 14200 7050 50  0000 L CNN
+F 2 "Resistor_SMD:R_Cat16-8" V 14175 7100 50  0001 C CNN
+F 3 "http://www.farnell.com/datasheets/1885635.pdf?_ga=2.1905073.1038136674.1585932994-1945507881.1583328620" H 13800 7100 50  0001 C CNN
+	1    13800 7100
+	1    0    0    -1
+$EndComp
