File: KiCad/Prototype/project.sch (KiCad schematic (older format))
At the start: 74 parts, among them J1 Barrel_Jack, J10 POT 2, J11 POT 3, J12 POT 4, J13 POT 5, J14 PRESSURE, J15 MIDI IN, J16 MIDI OUT, J17 POT 6, J18 POT 7, J19 POT 8, J2 USB_B, J20 TTL MIDI, J3 ICSP, J4 BANK 0..7, J5 BANK 8..15, J6 EXPRESSION, J7 SUSTAIN, J8 PD6/ADC9/SPEAKER, J9 POT 1, Q1 PMV48XP,215, SW1 RESET, U1 74LS75, U10 HCPL-0600, U2 LMV358, U3 AMS1117-5.0, U4 ATMEGA32U4-AU, U5 74HC138, U6 74HC138, U7 74HC238, U8 74HC238, U9 74HC04, Y1 16 Mhz

Commit message: minor tweaks
Parts:
- removed D3, D5: 1N914WT, footprints:D_SOD-323, symbol Diode:1N914WT
- added D3: BAV70, footprints:SOT-23, symbol Diode:BAV70
- added JP3: PULLUP, footprints:SolderJumper-3_P1.3mm_Bridged12_Pad1.0x1.5mm, symbol Jumper:Jumper_3_Bridged12
Connections:
- net +5V: now also JP3.3 (B)
- net ADC10: now also D3.3 (K)
- net GND: now also JP3.1 (A); no longer RN2.1 (R1.1), RN2.2 (R2.1), RN2.3 (R3.1), RN2.4 (R4.1), RN2.5 (R5.1), RN2.6 (R6.1)
- net at J6.T: now also D3.2 (A)
- net at J7.T, R10.1: now also D3.1 (A)
- new net: JP3.2 (C), RN2.1 (R1.1), RN2.2 (R2.1), RN2.3 (R3.1), RN2.4 (R4.1), RN2.5 (R5.1), RN2.6 (R6.1)
Changed lines of the file:
@@
 Wire Wire Line
 	11650 8850 11750 8850
-$Comp
-L Diode:1N914WT D3
-U 1 1 5EF15B1D
-P 11500 8650
-F 0 "D3" H 11500 8450 50  0000 R CNN
-F 1 "1N914WT" H 11750 8550 50  0000 R CNN
-F 2 "footprints:D_SOD-323" H 11500 8475 50  0001 C CNN
-F 3 "" H 11500 8650 50  0001 C CNN
-F 4 "C2128" H 11500 8650 50  0001 C CNN "LCSC"
-	1    11500 8650
-	1    0    0    1
-$EndComp
-Wire Wire Line
-	11650 8650 11700 8650
-Wire Wire Line
-	11700 8650 11700 8750
-Wire Wire Line
-	11700 8750 11750 8750
-Wire Wire Line
-	11350 8650 11050 8650
 Text Label 11050 8850 0    60   ~ 0
 AMUX1
-Text Label 11050 8650 0    60   ~ 0
-ADC10
 $Comp
 L project:GND #PWR043
@@
 	0    1    1    0
 $EndComp
-$Comp
-L Diode:1N914WT D5
-U 1 1 5F0071B8
-P 11550 7950
-F 0 "D5" H 11550 7750 50  0000 R CNN
-F 1 "1N914WT" H 11750 7850 50  0000 R CNN
-F 2 "footprints:D_SOD-323" H 11550 7775 50  0001 C CNN
-F 3 "" H 11550 7950 50  0001 C CNN
-F 4 "C2128" H 11550 7950 50  0001 C CNN "LCSC"
-	1    11550 7950
-	1    0    0    1
-$EndComp
-Wire Wire Line
-	11700 7950 11850 7950
 Wire Wire Line
 	11850 7650 11850 7950
@@
 	11400 7650 11050 7650
 Wire Wire Line
-	11400 7950 11050 7950
-Text Label 11050 7950 0    60   ~ 0
+	11350 8300 11050 8300
+Text Label 11050 8300 0    60   ~ 0
 ADC10
 Text Label 11050 7650 0    60   ~ 0
@@
 L project:GND #PWR049
 U 1 1 5F2725F4
-P 15350 9550
-F 0 "#PWR049" H 15350 9300 50  0001 C CNN
-F 1 "GND" H 15350 9400 50  0000 C CNN
-F 2 "" H 15350 9550 50  0001 C CNN
-F 3 "" H 15350 9550 50  0001 C CNN
-	1    15350 9550
+P 14250 9700
+F 0 "#PWR049" H 14250 9450 50  0001 C CNN
+F 1 "GND" H 14250 9550 50  0000 C CNN
+F 2 "" H 14250 9700 50  0001 C CNN
+F 3 "" H 14250 9700 50  0001 C CNN
+	1    14250 9700
 	1    0    0    -1
 $EndComp
@@
 Wire Wire Line
 	14750 9450 14850 9450
-Wire Wire Line
-	15350 9450 15350 9550
 Wire Wire Line
 	14850 9350 14850 9450
@@
 Wire Wire Line
 	15250 9350 15250 9450
-Connection ~ 15250 9450
-Wire Wire Line
-	15250 9450 15350 9450
 Wire Wire Line
 	13950 8650 13850 8650
@@
 ~HWB
 Connection ~ 4150 5250
+$Comp
+L Diode:BAV70 D3
+U 1 1 61730DDF
+P 11550 8300
+F 0 "D3" V 11504 8379 50  0000 L CNN
+F 1 "BAV70" V 11595 8379 50  0000 L CNN
+F 2 "footprints:SOT-23" H 11550 8300 50  0001 C CNN
+F 3 "https://assets.nexperia.com/documents/data-sheet/BAV70_SER.pdf" H 11550 8300 50  0001 C CNN
+F 4 "C68978" H 11550 8300 50  0001 C CNN "LCSC"
+	1    11550 8300
+	0    1    1    0
+$EndComp
+Wire Wire Line
+	11550 7950 11550 8000
+Wire Wire Line
+	11550 7950 11850 7950
+Wire Wire Line
+	11750 8750 11550 8750
+Wire Wire Line
+	11550 8750 11550 8600
+$Comp
+L Jumper:Jumper_3_Bridged12 JP3
+U 1 1 61923D82
+P 14250 9450
+F 0 "JP3" V 14296 9517 50  0000 L CNN
+F 1 "PULLUP" V 14205 9517 50  0000 L CNN
+F 2 "footprints:SolderJumper-3_P1.3mm_Bridged12_Pad1.0x1.5mm" H 14250 9450 50  0001 C CNN
+F 3 "~" H 14250 9450 50  0001 C CNN
+	1    14250 9450
+	0    -1   -1   0
+$EndComp
+$Comp
+L project:+5V #PWR025
+U 1 1 619586CA
+P 14250 9200
+F 0 "#PWR025" H 14250 9050 50  0001 C CNN
+F 1 "+5V" H 14250 9340 50  0000 C CNN
+F 2 "" H 14250 9200 50  0001 C CNN
+F 3 "" H 14250 9200 50  0001 C CNN
+	1    14250 9200
+	1    0    0    -1
+$EndComp
+Wire Wire Line
+	14400 9450 14750 9450
+Connection ~ 14750 9450
 $EndSCHEMATC

Commit message: Fix Kibot problems
Parts:
- U9: MOUSER 595-SN74HC04ANSRE4 -> (none)
Changed lines of the file:
@@
 F 1 "USB_B" H 4655 3026 50  0000 C CNN
 F 2 "footprints:USB_B_OST_USB-B1HSxx_Horizontal" H 4750 2600 50  0001 C CNN
-F 3 " ~" H 4750 2600 50  0001 C CNN
+F 3 "" H 4750 2600 50  0001 C CNN
 F 4 "490-UJ2-BH-1-TH" H 4600 2650 50  0001 C CNN "MOUSER"
 	1    4600 2650
@@
 F 2 "footprints:SOIC-14_3.9x8.7mm_P1.27mm" H 13050 2900 50  0001 C CNN
 F 3 "http://www.nxp.com/documents/data_sheet/74HC_HCT04.pdf" H 13050 2900 50  0001 C CNN
-F 4 "595-SN74HC04ANSRE4" H 13050 2900 50  0001 C CNN "MOUSER"
 	7    13050 2900
 	0    -1   -1   0

Commit message: trying again
Parts:
- U9: MOUSER 595-SN74HC04ANSRE4 -> (none)
Changed lines of the file:
@@
 F 2 "footprints:SOIC-14_3.9x8.7mm_P1.27mm" H 13050 3600 50  0001 C CNN
 F 3 "http://www.nxp.com/documents/data_sheet/74HC_HCT04.pdf" H 13050 3600 50  0001 C CNN
-F 4 "595-SN74HC04ANSRE4" H 13050 3600 50  0001 C CNN "MOUSER"
 	1    13050 3600
 	1    0    0    -1
@@
 F 2 "footprints:SOIC-14_3.9x8.7mm_P1.27mm" H 13650 3600 50  0001 C CNN
 F 3 "http://www.nxp.com/documents/data_sheet/74HC_HCT04.pdf" H 13650 3600 50  0001 C CNN
-F 4 "595-SN74HC04ANSRE4" H 13650 3600 50  0001 C CNN "MOUSER"
 	2    13650 3600
 	1    0    0    -1
